File: syzygy-mipi-adapter/syzygy-mipi-adapter.kicad_sch (KiCad schematic)
At the start: 67 parts, among them J1 Conn_02x06_Odd_Even, J10 501951-2230, J2 SYZYGY_STD, J3 Conn_01x02, J5 SM03B-SRSS-TB, J8 501951-2230, J9 501951-2230, Q1 DMG1024UV-7, Q2 DMG1024UV-7, U1 RP2350_80QFN, U10 PUSB3F96, U2 W25X20CLSNIG, U3 PUSB3F96, U4 PUSB3F96, U5 PUSB3F96, U6 PUSB3F96, U7 PUSB3F96, U8 PUSB3F96, U9 PUSB3F96, Y1 ABM8-272-T3

Commit message: fixes
Parts:
- added FID1, FID2, FID3, FID4, FID5, FID6, FID7, FID8: Fiducial, Fiducial:Fiducial_0.75mm_Mask1.5mm, symbol Mechanical:Fiducial
- added LOGO1: SYZYGY STD logo, SYZYGY:SYZYGY_STD_Logo, symbol MK11_PROG-rescue:TestPoint_Small-custom
- added LOGO2: SYZYGY logo, SYZYGY:SYZYGY_Logo, symbol MK11_PROG-rescue:TestPoint_Small-custom
- added R20: 10K, Resistor_SMD:R_0402_1005Metric, symbol Device:R_Small
- added R21: 0805, Resistor_SMD:R_0805_2012Metric_Pad1.20x1.40mm_HandSolder, symbol Device:R_Small
- J3: footprint Connector_PinHeader_1.27mm:PinHeader_1x03_P1.27mm_Vertical -> Connector_PinHeader_1.27mm:PinHeader_1x04_P1.27mm_Vertical; symbol Connector_Generic:Conn_01x03 -> Connector_Generic:Conn_01x04
- U2: value W25X20CLSNIG -> W25Q32JVSSIQ
Connections:
- net GND: now also J3.4 (Pin_4), R21.2
- net P3V3D: now also R20.1
- net at U1.56 (GPIO45_ADC5): now also R7.2
- net at U1.57 (GPIO46_ADC6): now also R20.2, R21.1; no longer R7.2
- no-connect marks 38 -> 37
Other:
- note added: "Estimate FPC internal skew to be 1mm for length matching purposes."
- note added: "PIO state machine I2C masters muxed to host I2C. Broadcast mode?"
- note added: "Potential divider configures I2C address of host I2C"
- note removed: "Muxed to host I2C. Broadcast mode?"
- moved on the sheet: H1, H2, H4, H6, R7

Commit message: Add USB connector and 3.3V regulator to Syzygy MIPI adapter
Parts:
- removed C44: 0.1uF, Capacitor_SMD:C_0402_1005Metric, symbol Device:C_Small
- removed J3: Conn_01x02, Connector_PinHeader_1.27mm:PinHeader_1x04_P1.27mm_Vertical, symbol Connector_Generic:Conn_01x04
- removed R13, R14, R15, R16, R17: 4.7K, Resistor_SMD:R_0402_1005Metric, symbol Device:R_Small
- removed R19: ~, Resistor_SMD:R_0402_1005Metric, symbol Device:R_Small
- removed R20: 10K, Resistor_SMD:R_0402_1005Metric, symbol Device:R_Small
- removed R21: 0805, Resistor_SMD:R_0805_2012Metric_Pad1.20x1.40mm_HandSolder, symbol Device:R_Small
- added C11, C12: 10u, Capacitor_SMD:C_0402_1005Metric, symbol Device:C
- added D1, D2: 1N5819WS, Diode_SMD:D_SOD-323, symbol Diode:1N5819WS
- added J3: USB_C_Receptacle_USB2.0_16P, Connector_USB:USB_C_Receptacle_HRO_TYPE-C-31-M-12, symbol Connector:USB_C_Receptacle_USB2.0_16P
- added LOGO3: OSHW logo, CUSTOM:OSHW_Dual_0.1_Scale_2140, symbol MK11_PROG-rescue:TestPoint_Small-custom
- added LOGO4: tinyAI logo, CUSTOM:tinyAI_logo, symbol MK11_PROG-rescue:TestPoint_Small-custom
- added R22, R25: 5.1K, Resistor_SMD:R_0402_1005Metric, symbol Device:R_Small
- added R23, R24: 56K, Resistor_SMD:R_0402_1005Metric, symbol Device:R_Small
- added R26: 10K, Resistor_SMD:R_0402_1005Metric, symbol Device:R_Small
- added R27: 15K, Resistor_SMD:R_0402_1005Metric, symbol Device:R_Small
- added RN1, RN2: 4.7K, Resistor_SMD:R_Array_Concave_4x0603, symbol Device:R_Pack04_Split
- added RN3, RN4: 4.7K, Resistor_SMD:R_Array_Concave_4x0603, symbol Device:R_Pack04
- added SW1: ~, CUSTOM:PTS820J25KSMTRLFS, symbol Switch:SW_Push
- added U11: NCP115AMX330TCG, Package_DFN_QFN:OnSemi_XDFN4-1EP_1.0x1.0mm_EP0.52x0.52mm, symbol Regulator_Linear:NCP115AMX120TCG
- R10: value 4.7K -> 10K; MPN (none) -> RC0402FR-0727RL; Manufacturer (none) -> YAGEO; Supplier (none) -> LCSC
- R11, R12: value 4.7K -> 56K; MPN (none) -> RC0402FR-0727RL; Manufacturer (none) -> YAGEO; Supplier (none) -> LCSC
- R7: value 100 -> 10K
- renumbered J5 to J4, J9 to J6, J8 to J6, J10 to J7, TP2 to TP1
Connections:
- net BYPASSn: now also RN2.3 (R3.1)
- net BYPASSn_3V3: now also RN2.4 (R4.1)
- net GND: now also R11.2, R12.2, C11.2, C12.2, J3.A1 (GND), J3.A12 (GND), J3.B1 (GND), J3.B12 (GND), J3.S1 (SHIELD), R22.2, R25.2, R27.2, SW1.1, SW1.SH1, SW1.SH2, U11.2 (GND), U11.5 (GND)
- net GPIO_HOST: now also RN2.1 (R1.1)
- net GPIO_HOST_3V3: now also RN2.2 (R2.1); no longer R12.2
- net P3V3D: now also C12.1, RN1.5 (R4.2), RN1.7 (R2.2), RN2.5 (R4.2), RN2.7 (R2.2), RN3.5 (R4.2), RN3.6 (R3.2), RN3.7 (R2.2), RN3.8 (R1.2), RN4.5 (R4.2), RN4.6 (R3.2), RN4.7 (R2.2), RN4.8 (R1.2), U11.1 (OUT); no longer J2.40 (+3.3V), R10.1, R11.1, R12.1, R18.1
- net P5VD: now also D2.2 (A); no longer C1.1, U1.64 (VREG_VIN)
- net PVIOD: now also RN1.6 (R3.2), RN1.8 (R1.2), RN2.6 (R3.2), RN2.8 (R1.2)
- net R_GA: now also R18.1; no longer R18.2
- net SCL0: now also RN4.2 (R2.1)
- net SCL1: now also RN3.4 (R4.1)
- net SCL2: now also RN3.2 (R2.1)
- net SCL3: now also RN4.4 (R4.1)
- net SCL_HOST: now also RN1.1 (R1.1)
- net SCL_HOST_3V3: now also RN1.2 (R2.1); no longer R10.2
- net SDA0: now also RN4.1 (R1.1)
- net SDA1: now also RN3.3 (R3.1)
- net SDA2: now also RN3.1 (R1.1)
- net SDA3: now also RN4.3 (R3.1)
- net SDA_HOST: now also RN1.3 (R3.1)
- net SDA_HOST_3V3: now also RN1.4 (R4.1); no longer R11.2
- net USB_D+: now reaches R5.1
- net USB_D+: now also J3.A6 (D+), J3.B6 (D+)
- net at U1.55 (GPIO44_ADC4): now also R10.2, R11.1
- net at R7.2, U1.56 (GPIO45_ADC5): now also R12.1
- net at U1.57 (GPIO46_ADC6): now also R26.2, R27.1
- net USB_D-: now reaches R6.1
- net USB_D-: now also J3.A7 (D-), J3.B7 (D-)
- net USB_BOOTn: no longer names the net of R8.1
- net USB_BOOTn: now also SW1.2
- new net: C1.1, C11.1, D1.1 (K), D2.1 (K), U1.64 (VREG_VIN), U11.3 (EN), U11.4 (IN)
- new net: J3.A5 (CC1), R22.1, R23.2
- new net: J3.B5 (CC2), R24.2, R25.1
- new net PVBUS: D1.2 (A), J3.A4 (VBUS), J3.A9 (VBUS), J3.B4 (VBUS), J3.B9 (VBUS), R23.1, R24.1, R26.1
- new net SZG_3V3: J2.40 (+3.3V), R10.1, R18.2
- no-connect marks 37 -> 36
Other:
- note added: "I2C masters muxed to host I2C"
- note added: "The ADC requires a 48MHz clock, which is provided by the USB PLL. Once the ADC has been used to measure R_GA:SZG_3V3 ratio, the ADC is disabled so that the USB PLL can be reused as a clock generator source."
- note added: "USB Boot"
- note added: "USB Connector"
- note added: "clock"
- note removed: "FPC"
- note removed: "Low: Host I2C addresses I2C mux High: Host I2C addresses IO expander / clock generator / mux control"
- note removed: "PIO state machine I2C masters muxed to host I2C. Broadcast mode?"
- note removed: "Potential divider configures I2C address of host I2C"
- moved on the sheet: C10, C33, C34, C36, C37, C39, C40, C41, C42, C43, C6, C7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

Commit message: Fix schematic ERC errors for Syzygy MIPI adapter
Parts:
- renumbered J6 to J8
Changed lines of the file:
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@@
 	)
 	(junction
+		(at 233.68 64.77)
+		(diameter 0)
+		(color 0 0 0 0)
+	)
+	(junction
 		(at 38.1 231.14)
 		(diameter 0)
@@
 	)
 	(junction
+		(at 26.67 46.99)
+		(diameter 0)
+		(color 0 0 0 0)
+	)
+	(junction
 		(at 250.19 60.96)
 		(diameter 0)
@@
 	(wire
 		(pts
-			(xy 229.87 64.77) (xy 240.03 64.77)
+			(xy 229.87 64.77) (xy 233.68 64.77)
 		)
 		(stroke
@@
 	(wire
 		(pts
+			(xy 233.68 64.77) (xy 240.03 64.77)
+		)
+		(stroke
+			(width 0)
+			(type default)
+		)
+	)
+	(wire
+		(pts
 			(xy 161.29 191.77) (xy 161.29 184.15)
 		)
@@
 	)
 	(symbol
+		(lib_id "power:PWR_FLAG")
+		(at 233.68 64.77 0)
+		(unit 1)
+		(exclude_from_sim no)
+		(in_bom yes)
+		(on_board yes)
+		(dnp no)
+		(fields_autoplaced yes)
+		(property "Reference" "#FLG06"
+			(at 233.68 62.865 0)
+			(effects
+				(font
+					(size 1.27 1.27)
+				)
+				(hide yes)
+			)
+		)
+		(property "Value" "PWR_FLAG"
+			(at 233.68 59.69 0)
+			(effects
+				(font
+					(size 1.27 1.27)
+				)
+				(hide yes)
+			)
+		)
+		(property "Footprint" ""
+			(at 233.68 64.77 0)
+			(effects
+				(font
+					(size 1.27 1.27)
+				)
+				(hide yes)
+			)
+		)
+		(property "Datasheet" "~"
+			(at 233.68 64.77 0)
+			(effects
+				(font
+					(size 1.27 1.27)
+				)
+				(hide yes)
+			)
+		)
+		(property "Description" "Special symbol for telling ERC where power comes from"
+			(at 233.68 64.77 0)
+			(effects
+				(font
+					(size 1.27 1.27)
+				)
+				(hide yes)
+			)
+		)
+		(pin "1"
+		)
+		(instances
+			(project ""
+				(path "/b75d5d5b-a423-49b6-bf7a-b3510d05dcb9"
+					(reference "#FLG06")
+					(unit 1)
+				)
+			)
+		)
+	)
+	(symbol
 		(lib_id "Device:C")
 		(at 88.9 62.23 0)
@@
 		(on_board yes)
 		(dnp no)
-		(property "Reference" "J6"
+		(property "Reference" "J8"
 			(at 372.11 145.542 0)
 			(effects
@@
 			(project "szg-mipi"
 				(path "/b75d5d5b-a423-49b6-bf7a-b3510d05dcb9"
-					(reference "J6")
+					(reference "J8")
 					(unit 1)
 				)
@@
 					(unit 1)
 				)
+			)
+		)
+	)
+	(symbol
+		(lib_id "power:PWR_FLAG")
+		(at 26.67 46.99 90)
+		(unit 1)
+		(exclude_from_sim no)
+		(in_bom yes)
+		(on_board yes)
+		(dnp no)
+		(fields_autoplaced yes)
+		(property "Reference" "#FLG05"
+			(at 24.765 46.99 0)
+			(effects
+				(font
+					(size 1.27 1.27)
+				)
+				(hide yes)
+			)
+		)
+		(property "Value" "PWR_FLAG"
+			(at 22.86 46.9899 90)
+			(effects
+				(font
+					(size 1.27 1.27)
+				)
+				(justify left)
+				(hide yes)
+			)
+		)
+		(property "Footprint" ""
+			(at 26.67 46.99 0)
+			(effects
+				(font
+					(size 1.27 1.27)
+				)
+				(hide yes)
+			)
+		)
+		(property "Datasheet" "~"
+			(at 26.67 46.99 0)
+			(effects
+				(font
+					(size 1.27 1.27)
+				)
+				(hide yes)
+			)
+		)
+		(property "Description" "Special symbol for telling ERC where power comes from"
+			(at 26.67 46.99 0)
+			(effects
+				(font
+					(size 1.27 1.27)
+				)
+				(hide yes)
+			)
+		)
+		(pin "1"
+		)
+		(instances
+			(project ""
+				(path "/b75d5d5b-a423-49b6-bf7a-b3510d05dcb9"
+					(reference "#FLG05")
+					(unit 1)
+				)

Commit message: Add USB connector and 3.3V regulator
Parts:
- RN1, RN2, RN3, RN4: footprint Resistor_SMD:R_Array_Concave_4x0603 -> Resistor_SMD:R_Array_Concave_4x0402
Connections:
- net BYPASSn: now also RN2.1 (R1.1); no longer RN2.3 (R3.1)
- net GPIO_HOST: now also RN2.3 (R3.1); no longer RN2.1 (R1.1)
- net P3V3D: now also RN1.6 (R3.2), RN1.8 (R1.2); no longer RN1.5 (R4.2), RN1.7 (R2.2)
- net PVIOD: now also RN1.5 (R4.2), RN1.7 (R2.2), RN2.6 (R3.2), RN2.8 (R1.2); no longer RN1.6 (R3.2), RN1.8 (R1.2), RN2.6 (R3.2), RN2.8 (R1.2)
- net SCL_HOST: now also RN1.4 (R4.1); no longer RN1.1 (R1.1)
- net SCL_HOST_3V3: now also RN1.1 (R1.1); no longer RN1.2 (R2.1)
- net SDA_HOST: now also RN1.2 (R2.1); no longer RN1.3 (R3.1)
- net SDA_HOST_3V3: now also RN1.3 (R3.1); no longer RN1.4 (R4.1)
Other:
- note added: "The ADC requires a 48MHz clock, provided by the USB PLL. Once the ADC has measured the R_GA:SZG_3V3 ratio, the ADC is disabled so that the USB PLL can be reused as a clock generator source."
- note removed: "The ADC requires a 48MHz clock, which is provided by the USB PLL. Once the ADC has been used to measure R_GA:SZG_3V3 ratio, the ADC is disabled so that the USB PLL can be reused as a clock generator source."
Changed lines of the file:
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@@
 		)
 	)
-	(text "The ADC requires a 48MHz clock, which is\nprovided by the USB PLL. Once the ADC has\nbeen used to measure R_GA:SZG_3V3 ratio,\nthe ADC is disabled so that the USB PLL\ncan be reused as a clock generator source."
+	(text "The ADC requires a 48MHz clock, provided\nby the USB PLL. Once the ADC has\nmeasured the R_GA:SZG_3V3 ratio,\nthe ADC is disabled so that the USB PLL\ncan be reused as a clock generator source."
 		(exclude_from_sim no)
 		(at 191.516 222.758 0)
@@
 			)
 		)
-		(property "Footprint" "Resistor_SMD:R_Array_Concave_4x0603"
+		(property "Footprint" "Resistor_SMD:R_Array_Concave_4x0402"
 			(at 254.508 232.41 90)
 			(effects
@@
 			)
 		)
-		(property "Footprint" "Resistor_SMD:R_Array_Concave_4x0603"
+		(property "Footprint" "Resistor_SMD:R_Array_Concave_4x0402"
 			(at 176.53 140.335 90)
 			(effects
@@
 		(lib_id "Device:R_Pack04_Split")
 		(at 256.54 153.67 0)
-		(unit 2)
+		(unit 1)
 		(exclude_from_sim no)
 		(in_bom yes)
@@
 			)
 		)
-		(property "Footprint" "Resistor_SMD:R_Array_Concave_4x0603"
+		(property "Footprint" "Resistor_SMD:R_Array_Concave_4x0402"
 			(at 254.508 153.67 90)
 			(effects
@@
 				(path "/b75d5d5b-a423-49b6-bf7a-b3510d05dcb9"
 					(reference "RN1")
-					(unit 2)
+					(unit 1)
 				)
 			)
@@
 		(lib_id "Device:R_Pack04_Split")
 		(at 256.54 180.34 0)
-		(unit 4)
+		(unit 3)
 		(exclude_from_sim no)
 		(in_bom yes)
@@
 			)
 		)
-		(property "Footprint" "Resistor_SMD:R_Array_Concave_4x0603"
+		(property "Footprint" "Resistor_SMD:R_Array_Concave_4x0402"
 			(at 254.508 180.34 90)
 			(effects
@@
 				(path "/b75d5d5b-a423-49b6-bf7a-b3510d05dcb9"
 					(reference "RN1")
-					(unit 4)
+					(unit 3)
 				)
 			)
@@
 			)
 		)
-		(property "Footprint" "Resistor_SMD:R_Array_Concave_4x0603"
+		(property "Footprint" "Resistor_SMD:R_Array_Concave_4x0402"
 			(at 254.508 205.74 90)
 			(effects
@@
 			)
 		)
-		(property "Footprint" "Resistor_SMD:R_Array_Concave_4x0603"
+		(property "Footprint" "Resistor_SMD:R_Array_Concave_4x0402"
 			(at 191.77 150.495 90)
 			(effects
@@
 		(lib_id "Device:R_Pack04_Split")
 		(at 278.13 153.67 0)
-		(unit 1)
+		(unit 4)
 		(exclude_from_sim no)
 		(in_bom yes)
@@
 			)
 		)
-		(property "Footprint" "Resistor_SMD:R_Array_Concave_4x0603"
+		(property "Footprint" "Resistor_SMD:R_Array_Concave_4x0402"
 			(at 276.098 153.67 90)
 			(effects
@@
 				(path "/b75d5d5b-a423-49b6-bf7a-b3510d05dcb9"
 					(reference "RN1")
-					(unit 1)
+					(unit 4)
 				)
 			)
@@
 		(lib_id "Device:R_Pack04_Split")
 		(at 278.13 232.41 0)
-		(unit 3)
+		(unit 1)
 		(exclude_from_sim no)
 		(in_bom yes)
@@
 			)
 		)
-		(property "Footprint" "Resistor_SMD:R_Array_Concave_4x0603"
+		(property "Footprint" "Resistor_SMD:R_Array_Concave_4x0402"
 			(at 276.098 232.41 90)
 			(effects
@@
 				(path "/b75d5d5b-a423-49b6-bf7a-b3510d05dcb9"
 					(reference "RN2")
-					(unit 3)
+					(unit 1)
 				)
 			)
@@
 		(lib_id "Device:R_Pack04_Split")
 		(at 278.13 205.74 0)
-		(unit 1)
+		(unit 3)
 		(exclude_from_sim no)
 		(in_bom yes)
@@
 			)
 		)
-		(property "Footprint" "Resistor_SMD:R_Array_Concave_4x0603"
+		(property "Footprint" "Resistor_SMD:R_Array_Concave_4x0402"
 			(at 276.098 205.74 90)
 			(effects
@@
 				(path "/b75d5d5b-a423-49b6-bf7a-b3510d05dcb9"
 					(reference "RN2")
-					(unit 1)
+					(unit 3)
 				)
 			)
@@
 		(lib_id "Device:R_Pack04_Split")
 		(at 278.13 180.34 0)
-		(unit 3)
+		(unit 2)
 		(exclude_from_sim no)
 		(in_bom yes)
@@
 			)
 		)
-		(property "Footprint" "Resistor_SMD:R_Array_Concave_4x0603"
+		(property "Footprint" "Resistor_SMD:R_Array_Concave_4x0402"
 			(at 276.098 180.34 90)
 			(effects
@@
 				(path "/b75d5d5b-a423-49b6-bf7a-b3510d05dcb9"
 					(reference "RN1")
-					(unit 3)
+					(unit 2)
 				)
 			)

Commit message: Add I2C test pads
Parts:
- added TP2, TP3, TP4, TP5, TP6, TP7: TestPoint, TestPoint:TestPoint_Pad_1.0x1.0mm, symbol Connector:TestPoint
Connections:
- net SCL0: now also TP3.1
- net SCL1: now also TP5.1
- net SCL2: now also TP7.1
- net SDA0: now also TP2.1
- net SDA1: now also TP4.1
- net SDA2: now also TP6.1
Other:
- moved on the sheet: RN3, RN4

Commit message: Sort out decoupling caps
Parts:
- added C13: 0.1u, Capacitor_SMD:C_0201_0603Metric, symbol Device:C
Connections:
- net GND: now also C13.2
- net P3V3D: now also C13.1
Changed lines of the file:
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@@
 	)
 	(junction
+		(at 190.5 49.53)
+		(diameter 0)
+		(color 0 0 0 0)
+	)
+	(junction
 		(at 52.07 154.94)
 		(diameter 0)
@@
 	)
 	(junction
+		(at 190.5 38.1)
+		(diameter 0)
+		(color 0 0 0 0)
+	)
+	(junction
 		(at 377.19 128.27)
 		(diameter 0)
@@
 	(wire
 		(pts
+			(xy 190.5 38.1) (xy 184.15 38.1)
+		)
+		(stroke
+			(width 0)
+			(type default)
+		)
+	)
+	(wire
+		(pts
 			(xy 153.67 140.97) (xy 190.5 140.97)
 		)
@@
 	(wire
 		(pts
-			(xy 184.15 49.53) (xy 184.15 50.8)
+			(xy 190.5 49.53) (xy 190.5 50.8)
 		)
 		(stroke
@@
 	(wire
 		(pts
+			(xy 190.5 46.99) (xy 190.5 49.53)
+		)
+		(stroke
+			(width 0)
+			(type default)
+		)
+	)
+	(wire
+		(pts
 			(xy 314.96 87.63) (xy 320.04 87.63)
 		)
@@
 	(wire
 		(pts
+			(xy 190.5 49.53) (xy 184.15 49.53)
+		)
+		(stroke
+			(width 0)
+			(type default)
+		)
+	)
+	(wire
+		(pts
 			(xy 177.8 49.53) (xy 184.15 49.53)
 		)
@@
 	(wire
 		(pts
+			(xy 190.5 39.37) (xy 190.5 38.1)
+		)
+		(stroke
+			(width 0)
+			(type default)
+		)
+	)
+	(wire
+		(pts
 			(xy 53.34 243.84) (xy 53.34 245.11)
 		)
@@
 	)
 	(symbol
+		(lib_id "Device:C")
+		(at 190.5 43.18 0)
+		(unit 1)
+		(exclude_from_sim no)
+		(in_bom yes)
+		(on_board yes)
+		(dnp no)
+		(property "Reference" "C13"
+			(at 190.5 41.275 0)
+			(effects
+				(font
+					(size 1.27 1.27)
+				)
+				(justify left)
+			)
+		)
+		(property "Value" "0.1u"
+			(at 191.135 45.72 0)
+			(effects
+				(font
+					(size 1.27 1.27)
+				)
+				(justify left)
+			)
+		)
+		(property "Footprint" "Capacitor_SMD:C_0201_0603Metric"
+			(at 191.4652 46.99 0)
+			(effects
+				(font
+					(size 1.27 1.27)
+				)
+				(hide yes)
+			)
+		)
+		(property "Datasheet" "~"
+			(at 190.5 43.18 0)
+			(effects
+				(font
+					(size 1.27 1.27)
+				)
+				(hide yes)
+			)
+		)
+		(property "Description" "Unpolarized capacitor"
+			(at 190.5 43.18 0)
+			(effects
+				(font
+					(size 1.27 1.27)
+				)
+				(hide yes)
+			)
+		)
+		(property "Digi-Key Part Number" ""
+			(at 190.5 43.18 0)
+			(effects
+				(font
+					(size 1.27 1.27)
+				)
+				(hide yes)
+			)
+		)
+		(property "MPN" "GRM155R71C104KA88J"
+			(at 190.5 43.18 0)
+			(effects
+				(font
+					(size 1.27 1.27)
+				)
+				(hide yes)
+			)
+		)
+		(property "Manufacturer" "Murata Electronics"
+			(at 190.5 43.18 0)
+			(effects
+				(font
+					(size 1.27 1.27)
+				)
+				(hide yes)
+			)
+		)
+		(property "Supplier" "Mouser"
+			(at 190.5 43.18 0)
+			(effects
+				(font
+					(size 1.27 1.27)
+				)
+				(hide yes)
+			)
+		)
+		(pin "1"
+		)
+		(pin "2"
+		)
+		(instances
+			(project "syzygy-mipi-adapter"
+				(path "/b75d5d5b-a423-49b6-bf7a-b3510d05dcb9"
+					(reference "C13")
+					(unit 1)
+				)
+			)
+		)
+	)
+	(symbol
 		(lib_id "power:GND")
 		(at 64.77 68.58 0)
@@
 	(symbol
 		(lib_id "power:VCC")
-		(at 184.15 38.1 0)
+		(at 190.5 38.1 0)
 		(unit 1)
 		(exclude_from_sim no)
@@
 		(dnp no)
 		(property "Reference" "#PWR018"
-			(at 184.15 41.91 0)
+			(at 190.5 41.91 0)
 			(effects
 				(font
@@
 		)
 		(property "Value" "P3V3D"
-			(at 184.531 33.7058 0)
+			(at 190.881 33.7058 0)
 			(effects
 				(font
@@
 		)
 		(property "Footprint" ""
-			(at 184.15 38.1 0)
+			(at 190.5 38.1 0)
 			(effects
 				(font
@@
 		)
 		(property "Datasheet" ""
-			(at 184.15 38.1 0)
+			(at 190.5 38.1 0)
 			(effects
 				(font
@@
 		)
 		(property "Description" "Power symbol creates a global label with name \"VCC\""
-			(at 184.15 38.1 0)
+			(at 190.5 38.1 0)
 			(effects
 				(font
@@
 	(symbol
 		(lib_id "power:GND")
-		(at 184.15 50.8 0)
+		(at 190.5 50.8 0)
 		(unit 1)
 		(exclude_from_sim no)
@@
 		(dnp no)
 		(property "Reference" "#PWR019"
-			(at 184.15 57.15 0)
+			(at 190.5 57.15 0)
 			(effects
 				(font
@@
 		)
 		(property "Value" "GND"
-			(at 184.277 55.1942 0)
+			(at 190.627 55.1942 0)
 			(effects
 				(font
@@
 		)
 		(property "Footprint" ""
-			(at 184.15 50.8 0)
+			(at 190.5 50.8 0)
 			(effects
 				(font
@@
 		)
 		(property "Datasheet" ""
-			(at 184.15 50.8 0)
+			(at 190.5 50.8 0)
 			(effects
 				(font
@@
 		)
 		(property "Description" "Power symbol creates a global label with name \"GND\" , ground"
-			(at 184.15 50.8 0)
+			(at 190.5 50.8 0)
 			(effects
 				(font

Commit message: Separate 3.3V rails for MSU vs Syzygy
Parts:
- added F1: MF-FSMF035X-2, Resistor_SMD:R_0603_1608Metric, symbol Device:Polyfuse_Small
Connections:
- net SZG_3V3 is gone; now on net P3V3D: J2.40 (+3.3V), R10.1, R18.2
- net P3V3D: no longer C10.1, C12.1, C13.1, C33.1, C34.1, C36.1, C37.1, C39.1, C40.1, C41.1, C42.1, C43.1, C9.1, R1.2, R2.2, R4.1, R9.2, U1.15 (IOVDD), U1.24 (IOVDD), U1.29 (IOVDD), U1.41 (IOVDD), U1.5 (IOVDD), U1.50 (IOVDD), U1.60 (IOVDD), U1.68 (USB_OTP_VDD), U1.69 (QSPI_IOVDD), U1.76 (IOVDD), U11.1 (OUT), U2.8 (VCC)
- net at C1.1, D1.1 (K), D2.1 (K)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: now also F1.1; no longer C11.1, U11.3 (EN), U11.4 (IN)
- new net: C11.1, F1.2, U11.3 (EN), U11.4 (IN)
- new net PMCUD: C10.1, C12.1, C13.1, C33.1, C34.1, C36.1, C37.1, C39.1, C40.1, C41.1, C42.1, C43.1, C9.1, R1.2, R2.2, R4.1, R9.2, U1.15 (IOVDD), U1.24 (IOVDD), U1.29 (IOVDD), U1.41 (IOVDD), U1.5 (IOVDD), U1.50 (IOVDD), U1.60 (IOVDD), U1.68 (USB_OTP_VDD), U1.69 (QSPI_IOVDD), U1.76 (IOVDD), U11.1 (OUT), U2.8 (VCC)
Other:
- note removed: "The ADC requires a 48MHz clock, provided by the USB PLL. Once the ADC has measured the R_GA:SZG_3V3 ratio, the ADC is disabled so that the USB PLL can be reused as a clock generator source."
- moved on the sheet: R11, R12, R18, R27
