File: syzygy-mipi-adapter/syzygy-mipi-adapter.kicad_sch (KiCad schematic)
At the start: 98 parts, among them J1 Conn_02x06_Odd_Even, J2 SYZYGY_STD, J3 USB_C_Receptacle_USB2.0_16P, J4 SM03B-SRSS-TB, J6 501951-2230, J7 501951-2230, J8 501951-2230, Q1 DMG1024UV-7, Q2 DMG1024UV-7, U1 RP2350_80QFN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

Commit message: Replace only 2.2u cap with 10u
Parts:
- C38: value 2.2u -> 10u
Changed lines of the file:
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@@
 			)
 		)
-		(property "Value" "2.2u"
+		(property "Value" "10u"
 			(at 164.465 78.74 0)
 			(effects

Commit message: Made tinyvision logo bigger
Parts:
- LOGO4: footprint CUSTOM:tinyAI_logo -> CUSTOM:tinyAI_4_5mm
Changed lines of the file:
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@@
 			)
 		)
-		(property "Footprint" "CUSTOM:tinyAI_logo"
+		(property "Footprint" "CUSTOM:tinyAI_4_5mm"
 			(at 367.03 240.284 0)
 			(effects
