File: syzygy-mipi-adapter/board/Rev1/syzygy-mipi-adapter.kicad_sch (KiCad schematic)
At the start: 98 parts, among them J1 Conn_02x06_Odd_Even, J2 SYZYGY_STD, J3 USB_C_Receptacle_USB2.0_16P, J4 SM03B-SRSS-TB, J6 501951-2230, J7 501951-2230, J8 501951-2230, Q1 DMG1024UV-7, Q2 DMG1024UV-7, U1 RP2350_80QFN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

Commit message: Consolidate footprints from several footprint libraries into CUSTOM.pretty
Parts:
- J6, J7, J8: footprint FPC:501951-2230 -> CUSTOM:501951-2230
- L1: footprint RP2350_60QFN_minimal:L_pol_2016 -> CUSTOM:L_pol_2016
- U1: footprint RP2350_60QFN_minimal:RP2350B_QFN-80_EP_10.573x10.573_Pitch0.4mm -> CUSTOM:RP2350B_QFN-80_EP_10.573x10.573_Pitch0.4mm
- U10, U3, U4, U5, U6, U7, U8, U9: footprint FPC:PUSB3F96X -> CUSTOM:PUSB3F96X
Changed lines of the file:
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@@
 			)
 		)
-		(property "Footprint" "FPC:PUSB3F96X"
+		(property "Footprint" "CUSTOM:PUSB3F96X"
 			(at 8.89 274.32 0)
 			(effects
@@
 			)
 		)
-		(property "Footprint" "FPC:PUSB3F96X"
+		(property "Footprint" "CUSTOM:PUSB3F96X"
 			(at 180.34 274.32 0)
 			(effects
@@
 			)
 		)
-		(property "Footprint" "FPC:PUSB3F96X"
+		(property "Footprint" "CUSTOM:PUSB3F96X"
 			(at 222.25 274.32 0)
 			(effects
@@
 			)
 		)
-		(property "Footprint" "FPC:501951-2230"
+		(property "Footprint" "CUSTOM:501951-2230"
 			(at 322.58 177.8 0)
 			(effects
@@
 			)
 		)
-		(property "Footprint" "FPC:501951-2230"
+		(property "Footprint" "CUSTOM:501951-2230"
 			(at 370.84 177.8 0)
 			(effects
@@
 			)
 		)
-		(property "Footprint" "RP2350_60QFN_minimal:L_pol_2016"
+		(property "Footprint" "CUSTOM:L_pol_2016"
 			(at 53.34 104.14 0)
 			(effects
@@
 			)
 		)
-		(property "Footprint" "RP2350_60QFN_minimal:RP2350B_QFN-80_EP_10.573x10.573_Pitch0.4mm"
+		(property "Footprint" "CUSTOM:RP2350B_QFN-80_EP_10.573x10.573_Pitch0.4mm"
 			(at 97.79 140.97 0)
 			(effects
@@
 			)
 		)
-		(property "Footprint" "FPC:PUSB3F96X"
+		(property "Footprint" "CUSTOM:PUSB3F96X"
 			(at 44.45 274.32 0)
 			(effects
@@
 			)
 		)
-		(property "Footprint" "FPC:PUSB3F96X"
+		(property "Footprint" "CUSTOM:PUSB3F96X"
 			(at 111.76 274.32 0)
 			(effects
@@
 			)
 		)
-		(property "Footprint" "FPC:PUSB3F96X"
+		(property "Footprint" "CUSTOM:PUSB3F96X"
 			(at 77.47 274.32 0)
 			(effects
@@
 			)
 		)
-		(property "Footprint" "FPC:501951-2230"
+		(property "Footprint" "CUSTOM:501951-2230"
 			(at 370.84 95.25 0)
 			(effects
@@
 			)
 		)
-		(property "Footprint" "FPC:PUSB3F96X"
+		(property "Footprint" "CUSTOM:PUSB3F96X"
 			(at 147.32 274.32 0)
 			(effects
@@
 			)
 		)
-		(property "Footprint" "FPC:PUSB3F96X"
+		(property "Footprint" "CUSTOM:PUSB3F96X"
 			(at 257.81 274.32 0)
 			(effects

Commit message: Fix issue #5 as described in that issue
Parts:
- removed R10: 10K, Resistor_SMD:R_0402_1005Metric, symbol Device:R_Small
- removed R11: 56K, Resistor_SMD:R_0402_1005Metric, symbol Device:R_Small
- renumbered J8 to J7, J7 to J8
Connections:
- net P3V3D: no longer R18.2
- net PMCUD: now also R18.2
- no-connect marks 34 -> 35
Other:
- moved on the sheet: R12, R18, R26, R27, R7
